File: PCB/Sandy_Top/Sandy_Top.kicad_sch (KiCad schematic)
At the start: 40 parts, among them J2 Conn_02x02_Top_Bottom, J3 Conn_02x02_Top_Bottom

Commit message: Topを仮配線。Midとの接続も一応確定
Parts:
- removed EXT_TR5: Conn_01x01, locallib:TestPoint_THTPad_D2.0mm_Drill1.0mm, symbol Connector_Generic:Conn_01x01
- removed H6, H8: MountingHole, locallib:MountingHole_2.2mm_M2_Pad_minimal, symbol Mechanical:MountingHole_Pad
- H1: renamed from H2; footprint locallib:MountingHole_2.2mm_M2_Pad_minimal -> locallib:MountingHole_1.8-2.2mm_M2_Pad_minimal
- H2: renamed from H3; footprint locallib:MountingHole_2.2mm_M2_Pad_minimal -> locallib:MountingHole_1.8-2.2mm_M2_Pad_minimal
- H3: renamed from H11; footprint locallib:MountingHole_2.2mm_M2_Pad_minimal -> locallib:MountingHole_1.8-2.2mm_M2_Pad_minimal
- H4: renamed from H12; footprint locallib:MountingHole_2.2mm_M2_Pad_minimal -> locallib:MountingHole_1.8-2.2mm_M2_Pad_minimal
- H5: renamed from H9; footprint locallib:MountingHole_2.2mm_M2_Pad_minimal -> locallib:MountingHole_1.8-2.2mm_M2_Pad_minimal
- H6: renamed from H10; footprint locallib:MountingHole_2.2mm_M2_Pad_minimal -> locallib:MountingHole_1.8-2.2mm_M2_Pad_minimal
- SW_;1, SW_[1: footprint locallib:Kailh_socket_ChocV2 -> locallib:Kailh_socket_ChocV2_small_#2pad
- renumbered J2 to #J22, J3 to #J33, D17 to D1, D18 to D2, D19 to D3, D16 to D4, D15 to D5, D20 to D6
Connections:
- net GND: now also H5.1; no longer H6.1
- net Top_col2: no longer #J33.2 (Pin_2), SW_T1.1
- net Top_col3: now also H2.1; no longer H1.1, SW_'1.1
- net Top_col4: now also H6.1, SW_'1.1, SW_T1.1; no longer H2.1
- net Top_row0: now also H1.1; no longer H3.1
- net Top_row1: now also D6.1 (K)
- net Top_row4: now also H3.1; no longer H5.1
- net Top_row5: no longer #J22.3 (Pin_3), D6.1 (K)
- no-connect marks 0 -> 2
Other:
- note added: "Col2 → Row4"
- note added: "Col3 → Row5"
- note added: "Topのピン数を減らすため場所を移動"
- moved on the sheet: D4, D6, H1, H2, H3, H4, H5, H6, SW_'1, SW_T1
