File: PCB/Sandy_Middle/Sandy_Middle.kicad_sch (KiCad schematic)
At the start: 79 parts, among them J1 Conn_02x02_Top_Bottom, J2 Conn_02x02_Top_Bottom, J3 Conn_02x02_Top_Bottom

Commit message: Topを仮配線。Midとの接続も一応確定
Parts:
- removed H_top_1, H_top_13, H_top_4, H_top_6, H_top_7, H_top_8, H_top_9: MountingHole, locallib:MountingHole_2.2mm_M2_Pad_minimal, symbol Mechanical:MountingHole_Pad
Connections:
- net GND: now also H12.1
- net Mid_GND: no longer H12.1
- net Mid_col2: now also SW_U1.1
- net Mid_col3: now also SW_H1.1
- net Mid_col4: no longer SW_H1.1, SW_U1.1
- net Mid_row1: no longer D9.1 (K)
- net Mid_row4: now also H_top_12.1
- net Mid_row5: now also D9.1 (K)
- net Mid_row6: no longer H_top_12.1
Other:
- note added: "Topのピン数を減らすためMidのスイッチを移動"
- moved on the sheet: D4, D9, H_top_10, H_top_11, H_top_12, H_top_2, H_top_3, H_top_5, SW_H1, SW_U1

Commit message: ピン調整
Parts:
- removed EXT_MC1, EXT_MC5, EXT_MR1: Conn_01x01, locallib:TestPoint_THTPad_D2.0mm_Drill1.0mm, symbol Connector_Generic:Conn_01x01
Connections:
- net Mid_GND is gone; now on net Mid_col4: H_top_10.1
- net GND: now also H_top_12.1; no longer H12.1
- net Mid_col0: no longer H1.1
- net Mid_col2: no longer H7.1
- net Mid_col3: no longer H3.1, H_top_2.1
- net Mid_col4: no longer H4.1, H_top_3.1
- net Mid_col6: no longer H6.1
- net Mid_row0: now also H_top_2.1; no longer H11.1, H_top_5.1
- net Mid_row1: no longer H2.1
- net Mid_row2: no longer H13.1
- net Mid_row3: no longer H15.1
- net Mid_row4: now also H_top_5.1; no longer H_top_12.1
- net Mid_row5: no longer H10.1
- net Mid_row6: no longer H5.1
- net Mid_col1: no longer names the net of H9.1
- net Mid_col5: no longer names the net of H8.1
