File: PCB/SandyLP_Middle/SandyLP_Middle.kicad_pcb (KiCad board)
At the start: 2 copper layers, 285 x 73.4 mm, 70 parts, among them J1 Conn_02x02_Top_Bottom, J2 Conn_02x02_Top_Bottom, J3 Conn_02x02_Top_Bottom

Commit message: とりあえずフットプリントを配置。左右孤立部などは考え中。
Parts:
- removed EXT_MC1, EXT_MC5, EXT_MR1, EXT_MR3, EXT_MR7, EXT_MR8: Conn_01x01, locallib:TestPoint_THTPad_D2.0mm_Drill1.0mm
- removed the H10 at (262.8, 39.1)
- removed the H12 at (303.2, 55.6)
- removed the H6 at (303.2, 24.1)
- removed H_top_1, H_top_13, H_top_4, H_top_6, H_top_7, H_top_8, H_top_9: MountingHole, locallib:MountingHole_2.2mm_M2_Pad_minimal
- removed J1, J2, J3: Conn_02x02_Top_Bottom, locallib:JST_SH_SM04B-SRSS-TB_1x04-1MP_P1.00mm_Horizontal_wCable_housing_spare_pin_courtyard
- added D1: D, locallib:D_SOD-123_Emphasized_Direction_Line, B.Cu at (125.8, -16.1)
- added D2: D, locallib:D_SOD-123_Emphasized_Direction_Line, B.Cu at (144.8, -15.4)
- added D3: D, locallib:D_SOD-123_Emphasized_Direction_Line, B.Cu at (163.9, -16.1)
- added D4: D, locallib:D_SOD-123_Emphasized_Direction_Line, B.Cu at (182.9, -15.4)
- added D5: D, locallib:D_SOD-123_Emphasized_Direction_Line, B.Cu at (144.8, 3.68)
- added D6: D, locallib:D_SOD-123_Emphasized_Direction_Line, B.Cu at (163.9, 2.95)
- added EXT_MR4: Conn_01x01, locallib:TestPoint_THTPad_D2.0mm_Drill1.0mm, F.Cu at (225.8, 66.3)
- added EXT_TC3: Conn_01x01, locallib:TestPoint_THTPad_D2.0mm_Drill1.0mm, B.Cu at (167.5, -20.1)
- added EXT_TC4: Conn_01x01, locallib:TestPoint_THTPad_D2.0mm_Drill1.0mm, B.Cu at (174.6, 8.45)
- added EXT_TR0: Conn_01x01, locallib:TestPoint_THTPad_D2.0mm_Drill1.0mm, B.Cu at (129.4, -18.9)
- added EXT_TR1: Conn_01x01, locallib:TestPoint_THTPad_D2.0mm_Drill1.0mm, B.Cu at (144.8, -1.08)
- added EXT_TR4: Conn_01x01, locallib:TestPoint_THTPad_D2.0mm_Drill1.0mm, B.Cu at (192.5, -16.6)
- added H1: MountingHole, locallib:MountingHole_1.8-2.2mm_M2_Pad_minimal, F.Cu at (140.1, -20.1)
- added H13: MountingHole, locallib:MountingHole_2.2mm_M2_Pad_minimal, F.Cu at (278.2, 43.7)
- added H14: MountingHole, locallib:MountingHole_2.2mm_M2_Pad_minimal, F.Cu at (297.3, 43.7)
- added H17: MountingHole, locallib:MountingHole_2.2mm_M2_Pad_minimal, F.Cu at (278.2, 55.6)
- added H18: MountingHole, locallib:MountingHole_2.2mm_M2_Pad_minimal, F.Cu at (297.3, 55.6)
- added H2: MountingHole, locallib:MountingHole_1.8-2.2mm_M2_Pad_minimal, F.Cu at (159.1, -14.2)
- added H3: MountingHole, locallib:MountingHole_1.8-2.2mm_M2_Pad_minimal, F.Cu at (178.2, -20.1)
- added H4: MountingHole, locallib:MountingHole_1.8-2.2mm_M2_Pad_minimal, F.Cu at (143.7, -4.65)
- added H6: MountingHole, locallib:MountingHole_2.2mm_M2_Pad_minimal, F.Cu at (163.9, 78.2)
- added H6: MountingHole, locallib:MountingHole_1.8-2.2mm_M2_Pad_minimal, F.Cu at (159.1, 4.88)
- added H7: MountingHole, locallib:MountingHole_2.2mm_M2_Pad_minimal, F.Cu at (142.5, 78.2)
- added REF**: ICON_Screw_Medium, locallib:ICON_Screw_Medium, F.Cu at (140.1, -13.6)
- added REF**: ICON_Screw_Medium, locallib:ICON_Screw_Medium, F.Cu at (159.0, -7.67)
- added REF**: ICON_Screw_Medium, locallib:ICON_Screw_Medium, F.Cu at (159.0, 3.63)
- added REF**: ICON_Screw_Medium, locallib:ICON_Screw_Medium, F.Cu at (147.0, -1.97)
- added REF**: ICON_Screw_Medium, locallib:ICON_Screw_Medium, F.Cu at (178.1, -13.6)
- added REF**: ICON_Screw_Medium, locallib:ICON_Screw_Medium, F.Cu at (170.8, -1.97)
- added SW_'1: SW_Push, locallib:Kailh_socket_ChocV2, F.Cu at (168.7, 4.88)
- added SW_;1: SW_Push, locallib:Kailh_socket_ChocV2_small_#2pad, F.Cu at (149.6, 4.88)
- added SW_T1: SW_Push, locallib:Kailh_socket_ChocV2, F.Cu at (187.7, -14.2)
- added SW_Y1: SW_Push, locallib:Kailh_socket_ChocV2, F.Cu at (168.7, -14.2)
- added SW_[1: SW_Push, locallib:Kailh_socket_ChocV2_small_#2pad, F.Cu at (130.6, -14.2)
- added SW_]1: SW_Push, locallib:Kailh_socket_ChocV2, F.Cu at (149.6, -14.2)
- Cutout1: footprint locallib:60_Outline-Sandy-DN0040-Mid -> locallib:SandyLP_outline_Mid
- H5: footprint locallib:MountingHole_2.2mm_M2_Pad_minimal -> locallib:MountingHole_1.8-2.2mm_M2_Pad_minimal
- SW_G1, SW_R1, SW_R4CNT_L1: footprint locallib:Kailh_socket_ChocV2 -> locallib:Kailh_socket_ChocV2_small_#2pad
- moved H_top_5 133.9 mm to (183.0, 43.7)
- moved H_top_10 115.0 mm to (163.9, 68.7)
- moved H3 105.1 mm to (202.0, 43.7)
- moved EXT_MR2 87.0 mm to (225.8, 80.6)
- moved H5 80.4 mm to (174.6, -4.65), turned to 0 degrees
- moved H_top_3 45.8 mm to (163.9, 49.6)
- moved H5 40.0 mm to (198.5, 59.2)
- moved H2 34.6 mm to (163.9, 43.7)
- moved H12 34.0 mm to (49.6, 42.5)
- moved H_top_2 27.3 mm to (144.9, 43.7)
- moved H8 24.1 mm to (184.2, 78.2)
- moved H_top_11 23.1 mm to (148.5, 59.2)
- moved H_top_12 23.1 mm to (179.4, 59.2)
- moved H1 21.7 mm to (125.8, 43.7)
- moved H11 19.3 mm to (30.6, 42.5)
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- renumbered H3 to H1, H16 to H10, H1 to H11, H2 to H12, H11 to H15, H9 to H16, H4 to H2, H7 to H3, H13 to H4, H8 to H5, H14 to H8, H15 to H9
Connections:
- D1 pad 1: Mid_row1 -> Mid_row0
- D11 pad 1: Mid_row8 -> Mid_row6
- D12 pad 1: Mid_row3 -> Mid_row2
- D13 pad 1: Mid_row3 -> Mid_row2
- D2 pad 1: Mid_row6 -> Mid_row4
- D3 pad 1: Mid_row1 -> Mid_row0
- D4 pad 1: Mid_row6 -> Mid_row4
- D5 pad 1: Mid_row1 -> Mid_row0
- D6 pad 1: Mid_row6 -> Mid_row4
- D7 pad 1: Mid_row7 -> Mid_row5
- D9 pad 1: Mid_row7 -> Mid_row5
- H1 pad 1: Mid_col3 -> Mid_row0
- H10 pad 1: Mid_row8 -> Mid_row2
- H12 pad 1: Mid_row1 -> Mid_row0
- H15 pad 1: Mid_row0 -> GND
- H16 pad 1: Mid_col1 -> Mid_row4
- H2 pad 1: Mid_col4 -> Mid_col3
- H3 pad 1: Mid_col2 -> Mid_row4
- H4 pad 1: Mid_row2 -> Mid_col2
- H5 pad 1: Mid_col5 -> GND
- H5 pad 1: Mid_row6 -> (no net)
- H8 pad 1: Mid_row7 -> Mid_row1
- H9 pad 1: Mid_row3 -> Mid_row6
- H_top_10 pad 1: Mid_GND -> Mid_col4
- H_top_12 pad 1: Mid_row6 -> GND
- H_top_2 pad 1: Mid_col3 -> Mid_row0
- H_top_3 pad 1: Mid_col4 -> Mid_col3
- H_top_5 pad 1: Mid_row0 -> Mid_row4
- SW_U1 pad 1: Mid_col4 -> Mid_col2
Routing:
- net Mid_col4: track 0.00 -> 63.9 mm, vias 0 -> 1
- net Mid_col3: track 0.00 -> 61.3 mm, vias 0 -> 2
- net Mid_row4: track 0.00 -> 50.9 mm
- net Mid_row0: track 0.00 -> 41.2 mm
- net Mid_row1: track 0.00 -> 26.5 mm
- net Net-(D3-A): track 0.00 -> 5.62 mm
- net Net-(D6-A): track 0.00 -> 5.48 mm
- net Net-(D1-A): track 0.00 -> 5.32 mm
- net Net-(D2-A): track 0.00 -> 5.11 mm
- net Net-(D5-A): track 0.00 -> 4.88 mm
- net Net-(D4-A): track 0.00 -> 4.88 mm
- added copper zone on B.Cu, net (none)
- added copper zone on F.Cu, net (none)
- removed copper zone on B.Cu, net Mid_GND
- removed copper zone on F.Cu, net Mid_GND
Other:
- board size 285 x 73.4 mm -> 113.1 x 56.3 mm
- board text added: "#SandyLP_kbd DN0010 Mid by @jpskenn"
- board text added: "#SandyLP_kbd DN0010 Top by @jpskenn"
- board text removed: "#Sandy_kbd DN0040, Mid by @jpskenn"
- board text removed: "Mid 1"
- board text removed: "Mid 2"

Commit message: ネジ位置調整
Parts:
- removed the H2 at (163.9, 43.7)
- removed the H6 at (163.9, 78.2)
- added REF**: ICON_Spacer, locallib:ICON_Spacer, F.Cu at (144.9, 62.7)
- added REF**: ICON_Spacer, locallib:ICON_Spacer, F.Cu at (164.0, 75.5)
- added REF**: ICON_Spacer, locallib:ICON_Spacer, F.Cu at (144.9, 50.8)
- added REF**: ICON_Screw_Medium, locallib:ICON_Screw_Medium, F.Cu at (132.9, 62.3)
- added REF**: ICON_Screw_Medium, locallib:ICON_Screw_Medium, F.Cu at (173.4, 86.1)
- added REF**: ICON_Spacer, locallib:ICON_Spacer, F.Cu at (183.0, 50.8)
- added REF**: ICON_Screw_Medium, locallib:ICON_Screw_Medium, F.Cu at (125.8, 50.4)
- added REF**: ICON_Screw_Medium, locallib:ICON_Screw_Medium, F.Cu at (201.9, 50.4)
- added REF**: ICON_Screw_Medium, locallib:ICON_Screw_Medium, F.Cu at (146.0, 81.4)
- added REF**: ICON_Screw_Medium, locallib:ICON_Screw_Medium, F.Cu at (194.8, 62.3)
- added REF**: ICON_Screw_Medium, locallib:ICON_Screw_Medium, F.Cu at (154.3, 86.1)
- added REF**: ICON_Screw_Medium, locallib:ICON_Screw_Medium, F.Cu at (180.5, 81.4)
- added REF**: ICON_Screw_Medium, locallib:ICON_Screw_Medium, B.Cu at (144.9, 62.3)
- added REF**: ICON_Nut & Washer, locallib:ICON_Nut & Washer, B.Cu at (133.0, 61.5)
- added REF**: ICON_Nut & Washer, locallib:ICON_Nut & Washer, B.Cu at (146.1, 80.6)
- added REF**: ICON_Nut & Washer, locallib:ICON_Nut & Washer, B.Cu at (194.8, 62.5)
- added REF**: ICON_Nut & Washer, locallib:ICON_Nut & Washer, B.Cu at (201.9, 50.5)
- added REF**: ICON_Nut & Washer, locallib:ICON_Nut & Washer, B.Cu at (154.3, 86.1)
- added REF**: ICON_Screw_Medium, locallib:ICON_Screw_Medium, B.Cu at (183.1, 62.3)
- added REF**: ICON_Screw_Medium, locallib:ICON_Screw_Medium, B.Cu at (145.0, 50.4)
- added REF**: ICON_Nut & Washer, locallib:ICON_Nut & Washer, B.Cu at (173.4, 86.1)
- added REF**: ICON_Spacer, locallib:ICON_Spacer, F.Cu at (183.0, 62.7)
- added REF**: ICON_Nut & Washer, locallib:ICON_Nut & Washer, B.Cu at (180.5, 81.4)
- added REF**: ICON_Screw_Medium, locallib:ICON_Screw_Medium, B.Cu at (183.1, 50.4)
- added REF**: ICON_Nut & Washer, locallib:ICON_Nut & Washer, B.Cu at (125.8, 50.5)
- added REF**: ICON_Spacer, locallib:ICON_Spacer, F.Cu at (163.9, 56.8)
- H1: footprint locallib:MountingHole_2.2mm_M2_Pad_minimal -> locallib:MountingHole_1.8-2.2mm_M2_Pad_minimal
- H10: renamed from H12; footprint locallib:MountingHole_2.2mm_M2_Pad_minimal -> locallib:MountingHole_1.8-2.2mm_M2_Pad_minimal
- H11: renamed from H13; footprint locallib:MountingHole_2.2mm_M2_Pad_minimal -> locallib:MountingHole_1.8-2.2mm_M2_Pad_minimal
- H12: renamed from H14; footprint locallib:MountingHole_2.2mm_M2_Pad_minimal -> locallib:MountingHole_1.8-2.2mm_M2_Pad_minimal
- H13: renamed from H15; footprint locallib:MountingHole_2.2mm_M2_Pad_minimal -> locallib:MountingHole_1.8-2.2mm_M2_Pad_minimal
- H14: renamed from H16; footprint locallib:MountingHole_2.2mm_M2_Pad_minimal -> locallib:MountingHole_1.8-2.2mm_M2_Pad_minimal
- H15: renamed from H17; footprint locallib:MountingHole_2.2mm_M2_Pad_minimal -> locallib:MountingHole_1.8-2.2mm_M2_Pad_minimal
- H16: renamed from H18; footprint locallib:MountingHole_2.2mm_M2_Pad_minimal -> locallib:MountingHole_1.8-2.2mm_M2_Pad_minimal
- H2: renamed from H3; footprint locallib:MountingHole_2.2mm_M2_Pad_minimal -> locallib:MountingHole_1.8-2.2mm_M2_Pad_minimal
- H3: renamed from H4; footprint locallib:MountingHole_2.2mm_M2_Pad_minimal -> locallib:MountingHole_1.8-2.2mm_M2_Pad_minimal
- H4: renamed from H5; footprint locallib:MountingHole_2.2mm_M2_Pad_minimal -> locallib:MountingHole_1.8-2.2mm_M2_Pad_minimal
- H5: renamed from H7; footprint locallib:MountingHole_2.2mm_M2_Pad_minimal -> locallib:MountingHole_1.8-2.2mm_M2_Pad_minimal
- H6: renamed from H8; footprint locallib:MountingHole_2.2mm_M2_Pad_minimal -> locallib:MountingHole_1.8-2.2mm_M2_Pad_minimal
- H7: renamed from H9; footprint locallib:MountingHole_2.2mm_M2_Pad_minimal -> locallib:MountingHole_1.8-2.2mm_M2_Pad_minimal
- H8: renamed from H10; footprint locallib:MountingHole_2.2mm_M2_Pad_minimal -> locallib:MountingHole_1.8-2.2mm_M2_Pad_minimal
- H9: renamed from H11; footprint locallib:MountingHole_2.2mm_M2_Pad_minimal -> locallib:MountingHole_1.8-2.2mm_M2_Pad_minimal
- H_top_1: renamed from H_top_2; footprint locallib:MountingHole_2.2mm_M2_Pad_minimal -> locallib:MountingHole_1.8-2.2mm_M2_Pad_minimal
- H_top_3: renamed from H_top_5; footprint locallib:MountingHole_2.2mm_M2_Pad_minimal -> locallib:MountingHole_1.8-2.2mm_M2_Pad_minimal
- H_top_4: renamed from H_top_11; footprint locallib:MountingHole_2.2mm_M2_Pad_minimal -> locallib:MountingHole_1.8-2.2mm_M2_Pad_minimal
- H_top_5: renamed from H_top_12; footprint locallib:MountingHole_2.2mm_M2_Pad_minimal -> locallib:MountingHole_1.8-2.2mm_M2_Pad_minimal
- moved D5 20.7 mm to (149.6, 23.8)
- moved EXT_TC3 20.7 mm to (172.3, 0.02)
- moved H1 20.7 mm to (144.9, 0.02)
- moved H3 20.7 mm to (183.0, 0.02)
- moved D1 20.7 mm to (130.6, 4.05)
- moved D2 20.7 mm to (149.6, 4.78)
- moved D3 20.7 mm to (168.7, 4.05)
- moved D4 20.7 mm to (187.7, 4.78)
- moved D6 20.7 mm to (168.7, 23.1)
- moved EXT_TC4 20.7 mm to (179.4, 28.6)
- moved EXT_TR0 20.7 mm to (134.2, 1.21)
- moved EXT_TR1 20.7 mm to (149.6, 19.1)
- moved EXT_TR4 20.7 mm to (197.3, 3.59)
- moved H2 20.7 mm to (163.9, 5.98)
- moved H4 20.7 mm to (148.5, 15.5)
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- renumbered H_top_3 to H_top_2, H_top_10 to H_top_6
Other:
- board text removed: "Mid 3"

Commit message: 不要なものを整理。
Other:
- board text removed: "to Base"
- board text removed: "to Top"

Commit message: 配線完了。ビア打ちまだ。
Parts:
- removed D1 (x2), D2 (x2), D5 (x2), D6 (x2): D, locallib:D_SOD-123_Emphasized_Direction_Line
- removed the D3 at (168.7, 4.05)
- removed the D4 at (187.7, 4.78)
- removed EXT_MC0, EXT_MC6, EXT_TC3, EXT_TC4, EXT_TR0, EXT_TR1, EXT_TR4: Conn_01x01, locallib:TestPoint_THTPad_D2.0mm_Drill1.0mm
- removed the H1 at (144.9, 0.02)
- removed H10, H11, H12, H13, H14, H15, H16, H9: MountingHole, locallib:MountingHole_1.8-2.2mm_M2_Pad_minimal
- removed the H2 at (163.9, 5.98)
- removed the H3 at (183.0, 0.02)
- removed the H4 at (148.5, 15.5)
- removed the H5 at (179.4, 15.5)
- removed the H6 at (163.9, 25.0)
- removed the REF** at (175.6, 18.2)
- removed the REF** at (144.9, 6.58)
- removed the REF** at (163.8, 12.5)
- removed the REF** at (163.8, 23.8)
- removed the REF** at (151.8, 18.2)
- removed the REF** at (182.9, 6.58)
- removed SW_'1, SW_BS1, SW_P1, SW_Q1, SW_T1, SW_TAB1, SW_Y1, SW_]1: SW_Push, locallib:Kailh_socket_ChocV2
- removed SW_;1, SW_[1: SW_Push, locallib:Kailh_socket_ChocV2_small_#2pad
- EXT_MR4: moved to B.Cu
- moved EXT_MR6 130.5 mm to (154.4, 78.2), turned to 0 degrees
- moved EXT_MR5 119.6 mm to (180.6, 66.3), turned to 0 degrees
- moved EXT_MR0 107.8 mm to (135.4, 47.2)
- moved EXT_MC4 70.9 mm to (156.8, 59.2), turned to 0 degrees
- moved EXT_MC2 68.8 mm to (171.1, 59.2), turned to 0 degrees
- moved EXT_MC3 56.9 mm to (163.9, 59.2), turned to 0 degrees
- moved EXT_MR2 52.4 mm to (173.5, 78.2), turned to 0 degrees
- moved EXT_MR4 38.4 mm to (192.5, 47.2), turned to 180 degrees
- moved D9 1.19 mm to (187.7, 67.5)
- moved D4 1.19 mm to (206.8, 48.4)
- moved REF** 0.54 mm to (144.7, 62.3)
Routing:
- net Mid_col2: track 0.00 -> 139.5 mm, vias 0 -> 2
- net Mid_row5: track 0.00 -> 71.3 mm
- net Mid_row2: track 0.00 -> 31.0 mm
- net Mid_row1: track 26.5 -> 53.3 mm, vias 0 -> 1
- net Mid_row6: track 0.00 -> 25.0 mm
- net Mid_row4: track 50.9 -> 28.1 mm
- net Mid_col3: track 61.3 -> 75.9 mm
- net Mid_col4: track 63.9 -> 57.3 mm
- net Net-(D6-A): track 5.48 -> 0.00 mm
- net Net-(D1-A): track 5.32 -> 0.00 mm
- net Net-(D2-A): track 5.11 -> 0.00 mm
- net Net-(D9-A): track 0.00 -> 4.88 mm
- net Net-(D5-A): track 4.88 -> 0.00 mm
- net Net-(D13-A): track 0.00 -> 4.88 mm
- net Net-(D12-A): track 0.00 -> 4.88 mm
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- added copper zone on B.Cu, net GND
- added copper zone on F.Cu, net GND
- removed copper zone on B.Cu, net (none)
- removed copper zone on F.Cu, net (none)
Other:
- board text removed: "#SandyLP_kbd DN0010 Top by @jpskenn"
