File: PCB/SandyLP_Middle/SandyLP_Middle.kicad_pcb (KiCad board)
At the start: 2 copper layers, 113.1 x 58.7 mm, 63 parts

Commit message: ネジ穴のアイコンを更新
Parts:
- added REF**: ICON_arrow_round_small, locallib:ICON_arrow_round_small, F.Cu at (166.3, 52.3)
- added REF**: ICON_arrow_round_small, locallib:ICON_arrow_round_small, F.Cu at (166.3, 71.1)
- REF** (x8): value ICON_Screw_Medium -> ICON_Screw_Long_Medium; footprint locallib:ICON_Screw_Medium -> locallib:ICON_Screw_Long_Medium
- moved REF** 5.68 mm to (133.1, 55.8), turned to 0 degrees
- moved REF** 5.68 mm to (146.2, 74.9), turned to 0 degrees
- moved REF** 5.41 mm to (194.8, 57.0), turned to 0 degrees
- moved REF** 5.29 mm to (173.6, 80.9), turned to 0 degrees
- moved REF** 5.28 mm to (154.3, 80.9), turned to 0 degrees
- moved REF** 5.28 mm to (180.5, 76.1), turned to 0 degrees
- moved REF** 4.22 mm to (201.9, 46.3), turned to 0 degrees
- moved REF** 4.22 mm to (125.8, 46.3), turned to 0 degrees
- moved REF** 2.24 mm to (125.8, 52.7)
- moved REF** 2.24 mm to (201.9, 52.7)
