File: PCB/SandyLP_Middle/SandyLP_Middle.kicad_sch (KiCad schematic)
At the start: 69 parts, among them J1 Conn_02x02_Top_Bottom, J2 Conn_02x02_Top_Bottom, J3 Conn_02x02_Top_Bottom

Commit message: とりあえずフットプリントを配置。左右孤立部などは考え中。
Parts:
- removed H10, H12, H5: MountingHole, locallib:MountingHole_2.2mm_M2_Pad_minimal, symbol Mechanical:MountingHole_Pad
- added H13, H14, H17, H18, H7: MountingHole, locallib:MountingHole_2.2mm_M2_Pad_minimal, symbol Mechanical:MountingHole_Pad
- SW_G1, SW_R1, SW_R4CNT_L1: footprint locallib:Kailh_socket_ChocV2 -> locallib:Kailh_socket_ChocV2_small_#2pad
- renumbered J1 to #J11, J2 to #J22, J3 to #J33, H3 to H1, H16 to H10, H1 to H11, H2 to H12, H11 to H15, H9 to H16, H4 to H2, H7 to H3, H13 to H4, H8 to H5, H14 to H8, H15 to H9
Connections:
- net GND: now also H15.1, H5.1, H17.1
- net Mid_col0: now also H11.1
- net Mid_col2: now also H4.1
- net Mid_col3: now also H2.1, H_top_3.1
- net Mid_col4: now also H6.1
- net Mid_col6: now also H13.1
- net Mid_row0: now also H1.1, H12.1, H14.1
- net Mid_row1: now also H8.1
- net Mid_row2: now also H10.1
- net Mid_row4: now also H16.1, H3.1, H18.1
- net Mid_row5: now also H7.1
- net Mid_row6: now also H9.1
- no-connect marks 2 -> 0
Other:
- moved on the sheet: H1, H10, H11, H12, H15, H16, H2, H3, H4, H5, H8, H9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

Commit message: ネジ位置調整
Parts:
- removed H2, H6: MountingHole, locallib:MountingHole_2.2mm_M2_Pad_minimal, symbol Mechanical:MountingHole_Pad
- H1: footprint locallib:MountingHole_2.2mm_M2_Pad_minimal -> locallib:MountingHole_1.8-2.2mm_M2_Pad_minimal
- H10: renamed from H12; footprint locallib:MountingHole_2.2mm_M2_Pad_minimal -> locallib:MountingHole_1.8-2.2mm_M2_Pad_minimal
- H11: renamed from H13; footprint locallib:MountingHole_2.2mm_M2_Pad_minimal -> locallib:MountingHole_1.8-2.2mm_M2_Pad_minimal
- H12: renamed from H14; footprint locallib:MountingHole_2.2mm_M2_Pad_minimal -> locallib:MountingHole_1.8-2.2mm_M2_Pad_minimal
- H13: renamed from H15; footprint locallib:MountingHole_2.2mm_M2_Pad_minimal -> locallib:MountingHole_1.8-2.2mm_M2_Pad_minimal
- H14: renamed from H16; footprint locallib:MountingHole_2.2mm_M2_Pad_minimal -> locallib:MountingHole_1.8-2.2mm_M2_Pad_minimal
- H15: renamed from H17; footprint locallib:MountingHole_2.2mm_M2_Pad_minimal -> locallib:MountingHole_1.8-2.2mm_M2_Pad_minimal
- H16: renamed from H18; footprint locallib:MountingHole_2.2mm_M2_Pad_minimal -> locallib:MountingHole_1.8-2.2mm_M2_Pad_minimal
- H2: renamed from H3; footprint locallib:MountingHole_2.2mm_M2_Pad_minimal -> locallib:MountingHole_1.8-2.2mm_M2_Pad_minimal
- H3: renamed from H4; footprint locallib:MountingHole_2.2mm_M2_Pad_minimal -> locallib:MountingHole_1.8-2.2mm_M2_Pad_minimal
- H4: renamed from H5; footprint locallib:MountingHole_2.2mm_M2_Pad_minimal -> locallib:MountingHole_1.8-2.2mm_M2_Pad_minimal
- H5: renamed from H7; footprint locallib:MountingHole_2.2mm_M2_Pad_minimal -> locallib:MountingHole_1.8-2.2mm_M2_Pad_minimal
- H6: renamed from H8; footprint locallib:MountingHole_2.2mm_M2_Pad_minimal -> locallib:MountingHole_1.8-2.2mm_M2_Pad_minimal
- H7: renamed from H9; footprint locallib:MountingHole_2.2mm_M2_Pad_minimal -> locallib:MountingHole_1.8-2.2mm_M2_Pad_minimal
- H8: renamed from H10; footprint locallib:MountingHole_2.2mm_M2_Pad_minimal -> locallib:MountingHole_1.8-2.2mm_M2_Pad_minimal
- H9: renamed from H11; footprint locallib:MountingHole_2.2mm_M2_Pad_minimal -> locallib:MountingHole_1.8-2.2mm_M2_Pad_minimal
- H_top_1: renamed from H_top_2; footprint locallib:MountingHole_2.2mm_M2_Pad_minimal -> locallib:MountingHole_1.8-2.2mm_M2_Pad_minimal
- H_top_3: renamed from H_top_5; footprint locallib:MountingHole_2.2mm_M2_Pad_minimal -> locallib:MountingHole_1.8-2.2mm_M2_Pad_minimal
- H_top_4: renamed from H_top_11; footprint locallib:MountingHole_2.2mm_M2_Pad_minimal -> locallib:MountingHole_1.8-2.2mm_M2_Pad_minimal
- H_top_5: renamed from H_top_12; footprint locallib:MountingHole_2.2mm_M2_Pad_minimal -> locallib:MountingHole_1.8-2.2mm_M2_Pad_minimal
- renumbered H_top_3 to H_top_2, H_top_10 to H_top_6
Other:
- note added: "このネジはTopとBottomの両方へ接続"
- moved on the sheet: H1, H3, H5, H7

Commit message: 配線完了。ビア打ちまだ。
Parts:
- removed D1, D2, D5, D6: D, locallib:D_SOD-123_Emphasized_Direction_Line, symbol Device:D
- removed EXT_MC0, EXT_MC6: Conn_01x01, locallib:TestPoint_THTPad_D2.0mm_Drill1.0mm, symbol Connector_Generic:Conn_01x01
- removed H10, H11, H12, H13, H14, H15, H16, H9: MountingHole, locallib:MountingHole_1.8-2.2mm_M2_Pad_minimal, symbol Mechanical:MountingHole_Pad
- removed SW_BS1, SW_P1, SW_Q1, SW_TAB1: SW_Push, locallib:Kailh_socket_ChocV2, symbol Switch:SW_Push

Commit message: ネジとソケットのパッドか近くはんだ付けが心配なため、パッドを少し小さくする。
Parts:
- SW_R4CNT_C1, SW_R4CNT_R1: footprint locallib:Kailh_socket_ChocV2 -> locallib:Kailh_socket_ChocV2_narrow_#2pad
Changed lines of the file:
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@@
 			)
 		)
-		(property "Footprint" "locallib:Kailh_socket_ChocV2"
+		(property "Footprint" "locallib:Kailh_socket_ChocV2_narrow_#2pad"
 			(at 175.26 103.505 0)
 			(effects
@@
 			)
 		)
-		(property "Footprint" "locallib:Kailh_socket_ChocV2"
+		(property "Footprint" "locallib:Kailh_socket_ChocV2_narrow_#2pad"
 			(at 142.24 103.505 0)
 			(effects
