File: PCB/SandyLP_Plate_Middle_Isolated_area/SandyLP_Plate_Middle_Isolated_area.kicad_sch (KiCad schematic)
At the start: 4 parts

Commit message: スイッチ穴をPTHに変更。
Parts:
- SW_BS1, SW_P1: footprint locallib:MX-Switch-Hole -> locallib:MXOnly-1U-Hotswap-guide-dummy
- SW_Q1, SW_TAB1: footprint locallib:MX-Switch-Hole -> locallib:MX-Switch-Hole-with-narrow-frame
Changed lines of the file:
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@@
 			)
 		)
-		(property "Footprint" "locallib:MX-Switch-Hole"
+		(property "Footprint" "locallib:MXOnly-1U-Hotswap-guide-dummy"
 			(at 257.81 40.005 0)
 			(effects
@@
 			)
 		)
-		(property "Footprint" "locallib:MX-Switch-Hole"
+		(property "Footprint" "locallib:MXOnly-1U-Hotswap-guide-dummy"
 			(at 241.3 40.005 0)
 			(effects
@@
 			)
 		)
-		(property "Footprint" "locallib:MX-Switch-Hole"
+		(property "Footprint" "locallib:MX-Switch-Hole-with-narrow-frame"
 			(at 59.69 40.005 0)
 			(effects
@@
 			)
 		)
-		(property "Footprint" "locallib:MX-Switch-Hole"
+		(property "Footprint" "locallib:MX-Switch-Hole-with-narrow-frame"
 			(at 43.18 40.005 0)
 			(effects
