File: PCB/SandyLP_Plate_Middle/SandyLP_Plate_Middle.kicad_pcb (KiCad board)
At the start: 2 copper layers, 113.1 x 58.7 mm, 8 parts

Commit message: スイッチ穴をPTHに変更。
Parts:
- SW_G1, SW_H1, SW_R1, SW_R4CNT_C1, SW_R4CNT_L1, SW_R4CNT_R1, SW_U1: footprint locallib:MX-Switch-Hole -> locallib:MX-Switch-Hole-with-narrow-frame
