File: PCB/SandyLP_Plate_Middle/SandyLP_Plate_Middle.kicad_sch (KiCad schematic)
At the start: 7 parts

Commit message: スイッチ穴をPTHに変更。
Parts:
- SW_G1, SW_H1, SW_R1, SW_R4CNT_C1, SW_R4CNT_L1, SW_R4CNT_R1, SW_U1: footprint locallib:MX-Switch-Hole -> locallib:MX-Switch-Hole-with-narrow-frame
Changed lines of the file:
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@@
 			)
 		)
-		(property "Footprint" "locallib:MX-Switch-Hole"
+		(property "Footprint" "locallib:MX-Switch-Hole-with-narrow-frame"
 			(at 158.75 71.755 0)
 			(effects
@@
 			)
 		)
-		(property "Footprint" "locallib:MX-Switch-Hole"
+		(property "Footprint" "locallib:MX-Switch-Hole-with-narrow-frame"
 			(at 109.22 40.005 0)
 			(effects
@@
 			)
 		)
-		(property "Footprint" "locallib:MX-Switch-Hole"
+		(property "Footprint" "locallib:MX-Switch-Hole-with-narrow-frame"
 			(at 175.26 103.505 0)
 			(effects
@@
 			)
 		)
-		(property "Footprint" "locallib:MX-Switch-Hole"
+		(property "Footprint" "locallib:MX-Switch-Hole-with-narrow-frame"
 			(at 125.73 40.64 0)
 			(effects
@@
 			)
 		)
-		(property "Footprint" "locallib:MX-Switch-Hole"
+		(property "Footprint" "locallib:MX-Switch-Hole-with-narrow-frame"
 			(at 125.73 71.755 0)
 			(effects
@@
 			)
 		)
-		(property "Footprint" "locallib:MX-Switch-Hole"
+		(property "Footprint" "locallib:MX-Switch-Hole-with-narrow-frame"
 			(at 125.73 103.505 0)
 			(effects
@@
 			)
 		)
-		(property "Footprint" "locallib:MX-Switch-Hole"
+		(property "Footprint" "locallib:MX-Switch-Hole-with-narrow-frame"
 			(at 142.24 103.505 0)
 			(effects
