File: PCB/SandyLP_Plate_Top/SandyLP_Plate_Top.kicad_pcb (KiCad board)
At the start: 2 copper layers, 285 x 56.6 mm, 38 parts

Commit message: 外形調整。スイッチ穴配置。
Parts:
- removed ?: , clipboard:1d23b097-72e0-487b-bec7-a328ee8b6ed7
- removed the REF** at (138.9, 27.0)
- removed the REF** at (167.5, 46.1)
- removed the REF** at (91.3, 27.0)
- removed the REF** at (62.7, 27.0)
- removed the REF** at (224.7, 27.0)
- removed the REF** at (129.4, 46.1)
- removed the REF** at (281.8, 27.0)
- removed the REF** at (148.5, 46.1)
- removed the REF** at (34.2, 27.0)
- removed the REF** at (253.2, 27.0)
- removed the REF** at (177.0, 27.0)
- removed the REF** at (167.5, 65.1)
- removed the REF** at (110.4, 27.0)
- removed the REF** at (148.5, 65.1)
- removed the REF** at (205.6, 27.0)
- removed the REF** at (186.6, 46.1)
- removed SW_'1, SW_1, SW_10, SW_2, SW_3, SW_4, SW_7, SW_8, SW_9, SW_;1, SW_ESC1, SW_INS1, SW_T1, SW_Y1: SW_Push, Jones.local:MXOnly-1U-Hotswap-guide-dummy
- REF**: footprint locallib:60_Outline-Sandy-DN0040-Plate-Top-outer-frame-only -> locallib:SandyLP_outline_Top
- SW_-1, SW_5, SW_6, SW_=1, SW_[1, SW_]1: footprint Jones.local:MXOnly-1U-Hotswap-guide-dummy -> locallib:MX-Switch-Hole
Other:
- board size 285 x 56.6 mm -> 74.9 x 39.4 mm
- board text added: "#SandyLP_kbd DN0010 Plate for Top by @jpskenn"
- board text removed: "#Sandy_kbd DN0040, Plate for Top by @jpskenn"

Commit message: スイッチ穴をPTHに変更。
Parts:
- SW_-1, SW_5, SW_6, SW_=1, SW_[1, SW_]1: footprint locallib:MX-Switch-Hole -> locallib:MX-Switch-Hole-with-narrow-frame
