File: PCB/SandyLP_Plate_Top/SandyLP_Plate_Top.kicad_pcb (KiCad board)
At the start: 2 copper layers, 74.9 x 39.4 mm, 7 parts

Commit message: オプションが無料になったのでJLCのマーキングを削除。その他シルク位置調整。
Other:
- board text added: "#SandyLP_kbd"
- board text added: "DN0010"
- board text added: "Plate for Top"
- board text added: "by @jpskenn"
- board text removed: "#SandyLP_kbd DN0010 Plate for Top by @jpskenn"
- board text removed: "Back Side"
- board text removed: "JLCJLCJLCJLC"
Changed lines of the file:
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@@
 			)
 		)
-		(attr through_hole)
+		(attr through_hole board_only exclude_from_pos_files exclude_from_bom)
 		(fp_line
 			(start -142.875 -38.1)
@@
 		(fp_arc
 			(start 18.425 1.164174)
-			(mid 19.01077 -0.250057)
+			(mid 19.010771 -0.250053)
 			(end 20.425 -0.835826)
 			(stroke
@@
 		(fp_arc
 			(start 18.44991 16.295746)
-			(mid 17.864148 17.709982)
+			(mid 17.864148 17.709986)
 			(end 16.44991 18.295746)
 			(stroke
@@
 		(fp_arc
 			(start 35.4625 -21.13133)
-			(mid 36.876724 -20.545545)
+			(mid 36.876689 -20.545539)
 			(end 37.4625 -19.13133)
 			(stroke
@@
 		)
 	)
-	(gr_text "Back Side"
-		(at 157.98031 36.528405 0)
-		(layer "B.SilkS" knockout)
-		(effects
-			(font
-				(size 2.2 2.2)
-				(thickness 0.225)
-				(italic yes)
-			)
-			(justify mirror)
-		)
-	)
-	(gr_text "JLCJLCJLCJLC"
-		(at 129.40531 18.278405 0)
+	(gr_text "DN0010"
+		(at 167.50531 18.497155 0)
 		(layer "B.SilkS")
 		(effects
 			(font
-				(size 1.5 1.5)
-				(thickness 0.3)
+				(size 1.2 1.2)
+				(thickness 0.15)
 			)
 			(justify mirror)
 		)
 	)
-	(gr_text "#SandyLP_kbd DN0010\nPlate for Top by @jpskenn"
-		(at 157.98031 17.478405 0)
+	(gr_text "by @jpskenn"
+		(at 129.40531 18.497155 0)
 		(layer "B.SilkS")
 		(effects
+			(font
+				(size 1.2 1.2)
+				(thickness 0.15)
+			)
+			(justify mirror)
+		)
+	)
+	(gr_text "Plate for Top"
+		(at 148.45531 18.497155 0)
+		(layer "B.SilkS")
+		(effects
+			(font
+				(size 1.2 1.2)
+				(thickness 0.15)
+			)
+			(justify mirror)
+		)
+	)
+	(gr_text "#SandyLP_kbd"
+		(at 186.55531 18.497155 0)
+		(layer "B.SilkS")
+		(effects
