File: PCB/SandyLP_Plate_Top/SandyLP_Plate_Top.kicad_sch (KiCad schematic)
At the start: 20 parts

Commit message: 外形調整。スイッチ穴配置。
Parts:
- removed SW_'1, SW_1, SW_10, SW_2, SW_3, SW_4, SW_7, SW_8, SW_9, SW_;1, SW_ESC1, SW_INS1, SW_T1, SW_Y1: SW_Push, Jones.local:MXOnly-1U-Hotswap-guide-dummy, symbol Switch:SW_Push
- SW_-1, SW_5, SW_6, SW_=1, SW_[1, SW_]1: footprint Jones.local:MXOnly-1U-Hotswap-guide-dummy -> locallib:MX-Switch-Hole

Commit message: スイッチ穴をPTHに変更。
Parts:
- SW_-1, SW_5, SW_6, SW_=1, SW_[1, SW_]1: footprint locallib:MX-Switch-Hole -> locallib:MX-Switch-Hole-with-narrow-frame
Changed lines of the file:
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@@
 			)
 		)
-		(property "Footprint" "locallib:MX-Switch-Hole"
+		(property "Footprint" "locallib:MX-Switch-Hole-with-narrow-frame"
 			(at 143.51 43.815 0)
 			(effects
@@
 			)
 		)
-		(property "Footprint" "locallib:MX-Switch-Hole"
+		(property "Footprint" "locallib:MX-Switch-Hole-with-narrow-frame"
 			(at 160.02 43.815 0)
 			(effects
@@
 			)
 		)
-		(property "Footprint" "locallib:MX-Switch-Hole"
+		(property "Footprint" "locallib:MX-Switch-Hole-with-narrow-frame"
 			(at 127 43.815 0)
 			(effects
@@
 			)
 		)
-		(property "Footprint" "locallib:MX-Switch-Hole"
+		(property "Footprint" "locallib:MX-Switch-Hole-with-narrow-frame"
 			(at 143.51 75.565 0)
 			(effects
@@
 			)
 		)
-		(property "Footprint" "locallib:MX-Switch-Hole"
+		(property "Footprint" "locallib:MX-Switch-Hole-with-narrow-frame"
 			(at 160.02 75.565 0)
 			(effects
@@
 			)
 		)
-		(property "Footprint" "locallib:MX-Switch-Hole"
+		(property "Footprint" "locallib:MX-Switch-Hole-with-narrow-frame"
 			(at 176.53 43.815 0)
 			(effects
