File: PCB/SandyLP_Plate_Bottom/SandyLP_Plate_Bottom.kicad_sch (KiCad schematic)
At the start: 45 parts

Commit message: 底面ロゴのサイズを大きく
Parts:
- removed LOGO1: Logo_Base, locallib:SandyLP_logo_w120, symbol Graphic:Logo_Open_Hardware_Small
Other:
- note removed: "LOGO"
Changed lines of the file:
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@@
-		)
-	)
-	(text "LOGO"
-		(exclude_from_sim no)
-		(at 245.745 19.05 0)
-		(effects
-			(font
-				(size 2.54 2.54)
-				(thickness 0.508)
-				(bold yes)
-			)
-			(justify left bottom)
 		)
 	)
@@
 					(unit 1)
 				)
-			)
-		)
-	)
-	(symbol
-		(lib_id "Graphic:Logo_Open_Hardware_Small")
-		(at 251.46 27.305 0)
-		(unit 1)
-		(exclude_from_sim yes)
-		(in_bom yes)
-		(on_board yes)
-		(dnp no)
-		(property "Reference" "LOGO1"
-			(at 257.7338 24.3586 0)
-			(effects
-				(font
-					(size 1.27 1.27)
-				)
-				(justify left)
-			)
-		)
-		(property "Value" "Logo_Base"
-			(at 257.7338 26.67 0)
-			(effects
-				(font
-					(size 1.27 1.27)
-				)
-				(justify left)
-			)
-		)
-		(property "Footprint" "locallib:SandyLP_logo_w120"
-			(at 251.46 27.305 0)
-			(effects
-				(font
-					(size 1.27 1.27)
-				)
-				(hide yes)
-			)
-		)
-		(property "Datasheet" "~"
-			(at 251.46 27.305 0)
-			(effects
-				(font
-					(size 1.27 1.27)
-				)
-				(hide yes)
-			)
-		)
-		(property "Description" ""
-			(at 251.46 27.305 0)
-			(effects
-				(font
-					(size 1.27 1.27)
-				)
-				(hide yes)
-			)
-		)
-		(property "Text" "@jpskenn"
-			(at 257.7338 28.9814 0)
-			(effects
-				(font
-					(size 1.27 1.27)
-				)
-				(justify left)
-			)
-		)
-		(instances
-			(project "Sandy_Base"
-				(path "/a99ab643-cdc7-4f8c-8088-c1f4faa914d1"
-					(reference "LOGO1")
-					(unit 1)
-				)
