File: PCB/SandyLP_Base/SandyLP_Base.kicad_pcb (KiCad board)
At the start: 2 copper layers, 275.5 x 80.3 mm, 229 parts, among them J1 Conn_01x10_Pin, J7 USB_C_Receptacle_USB2.0, J8 Conn_01x03, Q1 BSS138, SW1 BOOT, SW2 RESET, U1 NCP1117-3.3_SOT223, U2 RP2040, U3 W25Q128JVPIQ, Y1 12MHz

Commit message: ボトムプレートとの接続アイコンを修正
Parts:
- REF** (x11): value ICON_Nut -> ICON_Spacer; footprint locallib:ICON_Nut -> locallib:ICON_Spacer
- moved REF** 8.54 mm to (294.3, 48.8)
- moved REF** 3.35 mm to (209.1, 44.6)
- moved REF** 3.16 mm to (290.7, 111.3)
- moved REF** 3.15 mm to (63.3, 81.5)
- moved REF** 3.08 mm to (109.1, 44.6)
- moved REF** 3.08 mm to (254.4, 81.5)
- moved REF** 3.08 mm to (24.0, 48.8)
- moved REF** 2.75 mm to (209.7, 110.7)
- moved REF** 2.75 mm to (107.3, 110.7)
- moved REF** 2.63 mm to (155.4, 77.3)
- moved REF** 2.63 mm to (28.0, 111.3)

Commit message: オプションが無料になったのでJLCのマーキングを削除。その他シルク位置調整。
Other:
- board text removed: "JLCJLCJLCJLC"
Changed lines of the file:
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@@
 		(fp_arc
 			(start -0.378178 -1.358526)
-			(mid -0.787708 -1.474533)
+			(mid -0.787709 -1.474533)
 			(end -0.8 -1.9)
 			(stroke
@@
 		(fp_arc
 			(start -0.378178 -1.358526)
-			(mid -0.787708 -1.474533)
+			(mid -0.787709 -1.474533)
 			(end -0.8 -1.9)
 			(stroke
@@
 		(fp_arc
 			(start 0.7 3.345415)
-			(mid 0.662243 3.758488)
+			(mid 0.662244 3.758485)
 			(end 0.272339 3.9)
 			(stroke
@@
 		(fp_arc
 			(start 0.25 3.875)
-			(mid 0.26226 3.44949)
+			(mid 0.262251 3.449502)
 			(end 0.671822 3.333526)
 			(stroke
@@
 		(fp_arc
 			(start 0.7 3.345415)
-			(mid 0.662243 3.758488)
+			(mid 0.662244 3.758485)
 			(end 0.272339 3.9)
 			(stroke
@@
 		(fp_arc
 			(start 0.25 3.875)
-			(mid 0.26226 3.44949)
+			(mid 0.262251 3.449502)
 			(end 0.671822 3.333526)
 			(stroke
@@
 		(fp_arc
 			(start 0.7 3.345415)
-			(mid 0.662243 3.758488)
+			(mid 0.662244 3.758485)
 			(end 0.272339 3.9)
 			(stroke
@@
 		(fp_arc
 			(start 0.25 3.875)
-			(mid 0.26226 3.44949)
+			(mid 0.262251 3.449502)
 			(end 0.671822 3.333526)
 			(stroke
@@
 		(fp_arc
 			(start 0.7 3.345415)
-			(mid 0.662243 3.758488)
+			(mid 0.662244 3.758485)
 			(end 0.272339 3.9)
 			(stroke
@@
 		(fp_arc
 			(start 0.25 3.875)
-			(mid 0.26226 3.44949)
+			(mid 0.262251 3.449502)
 			(end 0.671822 3.333526)
 			(stroke
@@
 		(fp_arc
 			(start 0.7 3.345415)
-			(mid 0.662243 3.758488)
+			(mid 0.662244 3.758485)
 			(end 0.272339 3.9)
 			(stroke
@@
 		(fp_arc
 			(start 0.25 3.875)
-			(mid 0.26226 3.44949)
+			(mid 0.262251 3.449502)
 			(end 0.671822 3.333526)
 			(stroke
@@
 		(fp_arc
 			(start 0.7 3.345415)
-			(mid 0.662243 3.758488)
+			(mid 0.662244 3.758485)
 			(end 0.272339 3.9)
 			(stroke
@@
 		(fp_arc
 			(start 0.25 3.875)
-			(mid 0.26226 3.44949)
+			(mid 0.262251 3.449502)
 			(end 0.671822 3.333526)
 			(stroke
@@
 		(fp_arc
 			(start 0.7 3.345415)
-			(mid 0.662243 3.758488)
+			(mid 0.662244 3.758485)
 			(end 0.272339 3.9)
 			(stroke
@@
 		(fp_arc
 			(start 0.25 3.875)
-			(mid 0.26226 3.44949)
+			(mid 0.262251 3.449502)
 			(end 0.671822 3.333526)
 			(stroke
@@
 		(fp_arc
 			(start 0.7 3.345415)
-			(mid 0.662243 3.758488)
+			(mid 0.662244 3.758485)
 			(end 0.272339 3.9)
 			(stroke
@@
 		(fp_arc
 			(start 0.25 3.875)
-			(mid 0.26226 3.44949)
+			(mid 0.262251 3.449502)
 			(end 0.671822 3.333526)
 			(stroke
@@
 		(fp_arc
 			(start 0.7 3.345415)
-			(mid 0.662243 3.758488)
+			(mid 0.662244 3.758485)
 			(end 0.272339 3.9)
 			(stroke
@@
 		(fp_arc
 			(start 0.25 3.875)
-			(mid 0.26226 3.44949)
+			(mid 0.262251 3.449502)
 			(end 0.671822 3.333526)
 			(stroke
@@
 		(fp_arc
 			(start 0.7 3.345415)
-			(mid 0.662243 3.758488)
+			(mid 0.662244 3.758485)
 			(end 0.272339 3.9)
 			(stroke
@@
 		(fp_arc
 			(start 0.25 3.875)
-			(mid 0.26226 3.44949)
+			(mid 0.262251 3.449502)
 			(end 0.671822 3.333526)
 			(stroke
@@
 		(fp_arc
 			(start 0.7 3.345415)
-			(mid 0.662243 3.758488)
+			(mid 0.662244 3.758485)
 			(end 0.272339 3.9)
 			(stroke
@@
 		(fp_arc
 			(start 0.25 3.875)
-			(mid 0.26226 3.44949)
+			(mid 0.262251 3.449502)
 			(end 0.671822 3.333526)
 			(stroke
@@
 		)
 	)
-	(gr_text "JLCJLCJLCJLC"
-		(at 281.805529 36.528405 0)
-		(layer "B.SilkS")
-		(effects
-			(font
-				(size 1.5 1.5)
-			)
-			(justify left mirror)
-		)
-	)

Commit message: ロゴ更新
Parts:
- LOGO1: footprint locallib:SandyLP_logo_w60 -> locallib:SandyLP_logo_LP40_w60

Commit message: シルク追加。ロゴのフットプリント指定を修正。
Changed lines of the file:
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@@
 			)
 		)
+		(property "text" "RE1"
+			(at 3.45661 0 0)
+			(unlocked yes)
+			(layer "F.SilkS")
+			(effects
+				(font
+					(size 1 1)
+					(thickness 0.15)
+				)
+			)
+		)
 		(property ki_fp_filters "RotaryEncoder*Switch*")
 		(sheetname "ルート")
@@
 		(fp_arc
 			(start -0.378178 -1.358526)
-			(mid -0.787709 -1.474533)
+			(mid -0.787708 -1.474533)
 			(end -0.8 -1.9)
 			(stroke
@@
 		(sheetname "ルート")
 		(sheetfile "SandyLP_Base.kicad_sch")
-		(attr board_only exclude_from_pos_files exclude_from_bom)
 		(fp_poly
 			(pts
@@
 		(fp_arc
 			(start -0.378178 -1.358526)
-			(mid -0.787709 -1.474533)
+			(mid -0.787708 -1.474533)
 			(end -0.8 -1.9)
 			(stroke
@@
 		(tags "Murata Buzzer Beeper")
 		(property "Reference" "LS1"
-			(at 0 5.5 0)
+			(at 0 -5.45625 0)
 			(layer "B.SilkS")
-			(hide yes)
 			(effects
 				(font
@@
 		(tags "Murata Buzzer Beeper")
 		(property "Reference" "LS2"
-			(at 0 5.5 0)
+			(at -0.0875 -5.45625 0)
 			(layer "B.SilkS")
-			(hide yes)
 			(effects
 				(font
