File: PCB/SandyLP_Plate_Base_Center/SandyLP_Plate_Base_Center.kicad_pcb (KiCad board)
At the start: 2 copper layers, 103.6 x 39.8 mm, 8 parts

Commit message: プレートBase Center ゴムシート貼り付け指標
Other:
- board text added: "#SandyLP_kbd DN0020 Plate for Base-CNT by @jpskenn"
- board text removed: "#SandyLP_kbd"
- board text removed: "DN0011"
- board text removed: "Plate for Base-CNT"
- board text removed: "by @jpskenn"
Changed lines of the file:
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@@
 		(fp_arc
 			(start 88.34 37.54996)
-			(mid 86.925801 36.964171)
+			(mid 86.925765 36.964177)
 			(end 86.34 35.54996)
 			(stroke
@@
 		(fp_arc
 			(start 7.0125 37.785786)
-			(mid 5.598293 37.199991)
+			(mid 5.598297 37.199991)
 			(end 5.0125 35.785786)
 			(stroke
@@
 		(fp_arc
 			(start 88.34 37.54996)
-			(mid 86.92583 36.964142)
+			(mid 86.925795 36.964148)
 			(end 86.34 35.54996)
 			(stroke
@@
 		(fp_arc
 			(start 103.4 37.54996)
-			(mid 104.814228 38.135744)
+			(mid 104.814192 38.13575)
 			(end 105.4 39.54996)
 			(stroke
@@
 		(fp_arc
 			(start 107.4 56.54996)
-			(mid 105.985801 55.964171)
+			(mid 105.985765 55.964177)
 			(end 105.4 54.54996)
 			(stroke
@@
 		(fp_arc
 			(start 112.925 56.54996)
-			(mid 114.339228 57.135744)
+			(mid 114.339192 57.13575)
 			(end 114.925 58.54996)
 			(stroke
@@
 		(fp_arc
 			(start 116.925 75.62496)
-			(mid 115.510801 75.039171)
+			(mid 115.510765 75.039177)
 			(end 114.925 73.62496)
 			(stroke
@@
 		(fp_arc
 			(start 170.85 73.620746)
-			(mid 170.264168 75.034901)
+			(mid 170.264174 75.034936)
 			(end 168.85 75.620746)
 			(stroke
@@
 		(fp_arc
 			(start 180.35 39.471532)
-			(mid 180.935746 38.057268)
+			(mid 180.935752 38.057304)
 			(end 182.35 37.471532)
 			(stroke
@@
 		(fp_arc
 			(start 199.43 35.461532)
-			(mid 198.844173 36.875696)
+			(mid 198.844179 36.875731)
 			(end 197.43 37.461532)
 			(stroke
@@
 		(fp_arc
 			(start 95.845393 59.44996)
-			(mid 96.431187 58.035734)
+			(mid 96.431193 58.03577)
 			(end 97.845393 57.44996)
 			(stroke
@@
 		(fp_arc
 			(start 111.471875 57.44996)
-			(mid 112.886119 58.035735)
+			(mid 112.886084 58.035741)
 			(end 113.471875 59.44996)
 			(stroke
@@
 		(fp_arc
 			(start 172.228125 59.44996)
-			(mid 172.813927 58.035781)
+			(mid 172.813921 58.035746)
 			(end 174.228125 57.44996)
 			(stroke
@@
 		(fp_arc
 			(start 194.667351 95.28121)
-			(mid 194.081593 96.695464)
+			(mid 194.081587 96.695429)
 			(end 192.667351 97.28121)
 			(stroke
@@
 	)
 	(gr_rect
+		(start 113.779467 92.584744)
+		(end 130.01539 95.084744)
+		(stroke
+			(width 0.5)
+			(type default)
+		)
+		(fill none)
+		(layer "B.SilkS")
+	)
+	(gr_rect
+		(start 130.113063 96.373043)
+		(end 132.613063 110.227714)
+		(stroke
+			(width 0.5)
+			(type default)
+		)
+		(fill none)
+		(layer "B.SilkS")
+	)
+	(gr_rect
+		(start 187.381859 96.373042)
+		(end 189.881859 110.227713)
+		(stroke
+			(width 0.5)
+			(type default)
+		)
+		(fill none)
+		(layer "B.SilkS")
+	)
+	(gr_rect
+		(start 109.277108 96.373042)
+		(end 111.777108 110.227713)
+		(stroke
+			(width 0.5)
+			(type default)
+		)
+		(fill none)
+		(layer "B.SilkS")
+	)
+	(gr_rect
+		(start 189.979531 92.584744)
+		(end 206.215454 95.084744)
+		(stroke
+			(width 0.5)
+			(type default)
+		)
+		(fill none)
+		(layer "B.SilkS")
+	)
+	(gr_rect
+		(start 208.217814 96.373042)
+		(end 210.717814 110.227713)
+		(stroke
+			(width 0.5)
+			(type default)
+		)
+		(fill none)
+		(layer "B.SilkS")
+	)
+	(gr_rect
+		(start 109.909933 111.039447)
+		(end 210.084989 113.539447)
+		(stroke
+			(width 0.5)
+			(type default)
+		)
+		(fill none)
+		(layer "B.SilkS")
+	)
+	(gr_rect
 		(start 109.884845 21.24407)
 		(end 209.884845 121.24407)
@@
 		(layer "Eco1.User")
 	)
-	(gr_text "DN0011"
-		(at 179.047477 95.561309 0)
+	(gr_text "#SandyLP_kbd DN0020 Plate for Base-CNT by @jpskenn"
+		(at 159.997461 95.561309 0)
 		(layer "B.SilkS")
 		(effects
-			(font
-				(size 1 1)
-				(thickness 0.15)
-			)
-			(justify bottom mirror)
-		)
-	)
-	(gr_text "Plate for Base-CNT"
-		(at 140.947445 95.561309 0)
-		(layer "B.SilkS")
-		(effects
-			(font
-				(size 1 1)
-				(thickness 0.15)
-			)
-			(justify bottom mirror)
-		)
-	)
-	(gr_text "#SandyLP_kbd"
-		(at 200.478745 95.561309 0)
-		(layer "B.SilkS")
-		(effects
-			(font
-				(size 1 1)
-				(thickness 0.15)
-			)
-			(justify bottom mirror)
-		)
-	)
-	(gr_text "by @jpskenn"
-		(at 119.516177 95.561309 0)
-		(layer "B.SilkS")
-		(effects
